File: pcb/PCBcantik/FPGAforProg.brd (EAGLE design)
At the start: 100 x 80 mm, 1 part

Commit message: Update PCB
Parts:
- removed U$1: EPM7064STC44-10N, EPM7064STC44-10N:QFP80P1200X1200X120-44N
- added IC1: STM32F102C6T, micro-stm_v3:LQFP48
- added U1: 6SLX9TQG144, xilinx_devices:TQ144
Connections:
- removed net VCCINT: U$1.9
- removed net VCCINT_2: U$1.17
- removed net VCCINT_3: U$1.29
- removed net VCCINT_4: U$1.41
- new net GND: U1.P108, U1.P113, U1.P13, U1.P130, U1.P136, U1.P25, U1.P3, U1.P49, U1.P54, U1.P68, U1.P77, U1.P91, U1.P96
- new net N$1: IC1.1, U1.P1
- new net VDD: IC1.24, IC1.36, IC1.48
- new net VDDA: IC1.9
- new net VSS: IC1.23, IC1.35, IC1.47
- new net VSSA: IC1.8
Changed lines of the file:
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@@
 </autorouter>
 <elements>
-<element name="U$1" library="EPM7064STC44-10N" package="QFP80P1200X1200X120-44N" value="EPM7064STC44-10N" x="49.53" y="46.99">
-<attribute name="AVAILABILITY" value="Good" x="49.53" y="46.99" size="1.778" layer="27" display="off"/>
-<attribute name="DESCRIPTION" value=" IC: CPLD; SMD; TQFP44; Series: Max 7000; Amount of macr " x="49.53" y="46.99" size="1.778" layer="27" display="off"/>
-<attribute name="MF" value="Altera" x="49.53" y="46.99" size="1.778" layer="27" display="off"/>
-<attribute name="MP" value="EPM7064STC44-10N" x="49.53" y="46.99" size="1.778" layer="27" display="off"/>
-<attribute name="PACKAGE" value="TQFP-44 Altera" x="49.53" y="46.99" size="1.778" layer="27" display="off"/>
-<attribute name="PRICE" value="8.09 USD" x="49.53" y="46.99" size="1.778" layer="27" display="off"/>
-</element>
+<element name="U1" library="xilinx_devices" package="TQ144" value="6SLX9TQG144" x="48.26" y="39.37"/>
+<element name="IC1" library="micro-stm_v3" package="LQFP48" value="STM32F102C6T" x="15.24" y="57.15" rot="R270"/>
 </elements>
 <signals>
-<signal name="VCCINT_2">
-<contactref element="U$1" pad="17"/>
+<signal name="GND">
+<contactref element="U1" pad="P108"/>
+<contactref element="U1" pad="P113"/>
+<contactref element="U1" pad="P13"/>
+<contactref element="U1" pad="P130"/>
+<contactref element="U1" pad="P136"/>
+<contactref element="U1" pad="P25"/>
+<contactref element="U1" pad="P3"/>
+<contactref element="U1" pad="P49"/>
+<contactref element="U1" pad="P54"/>
+<contactref element="U1" pad="P68"/>
+<contactref element="U1" pad="P77"/>
+<contactref element="U1" pad="P91"/>
+<contactref element="U1" pad="P96"/>
+<wire x1="55.01" y1="50.47" x2="59.36" y2="48.12" width="0" layer="19" extent="1-1"/>
+<wire x1="59.36" y1="42.12" x2="59.36" y2="48.12" width="0" layer="19" extent="1-1"/>
+<wire x1="59.36" y1="39.62" x2="59.36" y2="42.12" width="0" layer="19" extent="1-1"/>
+<wire x1="59.36" y1="32.62" x2="59.36" y2="39.62" width="0" layer="19" extent="1-1"/>
+<wire x1="55.01" y1="28.27" x2="59.36" y2="32.62" width="0" layer="19" extent="1-1"/>
+<wire x1="48.01" y1="28.27" x2="55.01" y2="28.27" width="0" layer="19" extent="1-1"/>
+<wire x1="45.51" y1="28.27" x2="48.01" y2="28.27" width="0" layer="19" extent="1-1"/>
+<wire x1="46.51" y1="50.47" x2="55.01" y2="50.47" width="0" layer="19" extent="1-1"/>
+<wire x1="43.51" y1="50.47" x2="46.51" y2="50.47" width="0" layer="19" extent="1-1"/>
+<wire x1="37.16" y1="47.12" x2="43.51" y2="50.47" width="0" layer="19" extent="1-1"/>
+<wire x1="37.16" y1="42.12" x2="37.16" y2="47.12" width="0" layer="19" extent="1-1"/>
+<wire x1="37.16" y1="36.12" x2="37.16" y2="42.12" width="0" layer="19" extent="1-1"/>
 </signal>
-<signal name="VCCINT_3">
-<contactref element="U$1" pad="29"/>
+<signal name="VDDA">
+<contactref element="IC1" pad="9"/>
 </signal>
-<signal name="VCCINT_4">
-<contactref element="U$1" pad="41"/>
+<signal name="VSSA">
+<contactref element="IC1" pad="8"/>
 </signal>
-<signal name="VCCINT">
-<contactref element="U$1" pad="9"/>
+<signal name="VDD">
+<contactref element="IC1" pad="24"/>
+<contactref element="IC1" pad="36"/>
+<contactref element="IC1" pad="48"/>
+<wire x1="19.49" y1="59.9" x2="17.99" y2="52.9" width="0" layer="19" extent="1-1"/>
+<wire x1="12.49" y1="61.4" x2="19.49" y2="59.9" width="0" layer="19" extent="1-1"/>
+</signal>
+<signal name="VSS">
+<contactref element="IC1" pad="23"/>
+<contactref element="IC1" pad="35"/>
+<contactref element="IC1" pad="47"/>
+<wire x1="19.49" y1="59.4" x2="17.49" y2="52.9" width="0" layer="19" extent="1-1"/>
+<wire x1="12.99" y1="61.4" x2="19.49" y2="59.4" width="0" layer="19" extent="1-1"/>
+</signal>
+<signal name="N$1">
+<contactref element="IC1" pad="1"/>
+<contactref element="U1" pad="P1"/>
+<wire x1="10.99" y1="59.9" x2="37.16" y2="48.12" width="0" layer="19" extent="1-1"/>
 </signal>
 </signals>
