File: pcb/PCBcantik/FPGAforProg.sch (EAGLE design)
At the start: 1 part

Commit message: Update PCB
Parts:
- removed U$1: EPM7064STC44-10N, EPM7064STC44-10N:EPM7064STC44-10N
- added IC1: STM32F051R4T, micro-stm_v3:STM32F051R4T
- added U1: 6SLX9TQG144, xilinx_devices:6SLX9TQG144
Other:
- note removed: "Ini FPGA"
Changed lines of the file:
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@@
 </classes>
 <parts>
-<part name="U$1" library="EPM7064STC44-10N" deviceset="EPM7064STC44-10N" device=""/>
+<part name="U1" library="xilinx_devices" deviceset="6SLX9TQG144" device=""/>
+<part name="IC1" library="micro-stm_v3" deviceset="STM32F051R*T" device="" technology="4"/>
 </parts>
 <sheets>
 <sheet>
 <plain>
-<text x="43.18" y="22.86" size="1.778" layer="91">Ini FPGA</text>
 </plain>
 <instances>
-<instance part="U$1" gate="A" x="58.42" y="50.8"/>
+<instance part="U1" gate="B0" x="-5.08" y="53.34"/>
+<instance part="U1" gate="B1" x="53.34" y="55.88"/>
+<instance part="U1" gate="B2" x="114.3" y="53.34"/>
+<instance part="U1" gate="B3" x="177.8" y="53.34"/>
+<instance part="U1" gate="BNA" x="58.42" y="134.62"/>
+<instance part="U1" gate="BVCCAUX" x="139.7" y="129.54"/>
+<instance part="U1" gate="BVCCINT" x="78.74" y="-7.62"/>
+<instance part="IC1" gate="MCU" x="243.84" y="60.96"/>
 </instances>
 <busses>
